File: PCB/PiicoDev OLED SSD1306.kicad_sch (KiCad schematic)
At the start: 30 parts, among them J1 , J2 , J3 Conn_PiicoDev_header_01x04_Ma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, SW1 SW_DIP_x01, U2 Display_Graphic_OLED_SSD1306_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

Commit message: rotate ASW
Connections:
- net +3V3: now also SW1.2; no longer SW1.1
- net SA0: now also SW1.1; no longer SW1.2
Changed lines of the file:
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@@
     )
   )
-  (symbol (lib_id "Switch:SW_DIP_x01") (at 171.45 62.23 270) (unit 1)
+  (symbol (lib_id "Switch:SW_DIP_x01") (at 171.45 62.23 270) (mirror x) (unit 1)
     (in_bom yes) (on_board yes)
-    (property "Reference" "SW1" (id 0) (at 174.752 61.0616 90)
+    (property "Reference" "SW1" (id 0) (at 174.752 63.3984 90)
       (effects (font (size 1.27 1.27)) (justify left))
     )
-    (property "Value" "SW_DIP_x01" (id 1) (at 174.752 63.373 90)
+    (property "Value" "SW_DIP_x01" (id 1) (at 174.752 61.087 90)
       (effects (font (size 1.27 1.27)) (justify left))
     )

Commit message: update to v13 with reduced paste on OLED
Parts:
- removed H3, H4: MountingHole, PiicoDev OLED SSD1306:OLED_SSD1306_Hole, symbol Mechanical:MountingHole
- U2: footprint Display:OLED-128O064D -> CoreElectronics_Components:OLED-128O064D_reduced_paste
Changed lines of the file:
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@@
     (property "Reference" "U2" (id 0) (at 205.74 49.53 0))
     (property "Value" "Display_Graphic_OLED_SSD1306_30-Pin" (id 1) (at 246.38 125.73 0))
-    (property "Footprint" "Display:OLED-128O064D" (id 2) (at 215.9 107.95 0)
+    (property "Footprint" "CoreElectronics_Components:OLED-128O064D_reduced_paste" (id 2) (at 215.9 107.95 0)
       (effects (font (size 1.27 1.27)) hide)
     )
@@
     (pin "1")
   )
-  (symbol (lib_id "Mechanical:MountingHole") (at 162.56 189.23 0) (unit 1)
-    (in_bom yes) (on_board yes)
-    (property "Reference" "H3" (id 0) (at 165.1 188.0616 0)
-      (effects (font (size 1.27 1.27)) (justify left) hide)
-    )
-    (property "Value" "MountingHole" (id 1) (at 165.1 190.373 0)
-      (effects (font (size 1.27 1.27)) (justify left) hide)
-    )
-    (property "Footprint" "PiicoDev OLED SSD1306:OLED_SSD1306_Hole" (id 2) (at 162.56 189.23 0)
-      (effects (font (size 1.27 1.27)) hide)
-    )
-    (property "Datasheet" "~" (id 3) (at 162.56 189.23 0)
-      (effects (font (size 1.27 1.27)) hide)
-    )
-  )
-  (symbol (lib_id "Mechanical:MountingHole") (at 162.56 194.31 0) (unit 1)
-    (in_bom yes) (on_board yes)
-    (property "Reference" "H4" (id 0) (at 165.1 193.1416 0)
-      (effects (font (size 1.27 1.27)) (justify left) hide)
-    )
-    (property "Value" "MountingHole" (id 1) (at 165.1 195.453 0)
-      (effects (font (size 1.27 1.27)) (justify left) hide)
-    )
-    (property "Footprint" "PiicoDev OLED SSD1306:OLED_SSD1306_Hole" (id 2) (at 162.56 194.31 0)
-      (effects (font (size 1.27 1.27)) hide)
-    )
-    (property "Datasheet" "~" (id 3) (at 162.56 194.31 0)
-      (effects (font (size 1.27 1.27)) hide)
-    )
-  )
   (symbol (lib_id "Switch:SW_DIP_x01") (at 171.45 62.23 270) (mirror x) (unit 1)
     (in_bom yes) (on_board yes)
@@
       (reference "H2") (unit 1) (value "MountingHole") (footprint "CoreElectronics_Components:MountingHole_2.7mm_M2.5_PadClearance_1.2")
     )
-    (path "/00000000-0000-0000-0000-000060ef2d1b"
-      (reference "H3") (unit 1) (value "MountingHole") (footprint "PiicoDev OLED SSD1306:OLED_SSD1306_Hole")
-    )
-    (path "/00000000-0000-0000-0000-000060ef31e9"
-      (reference "H4") (unit 1) (value "MountingHole") (footprint "PiicoDev OLED SSD1306:OLED_SSD1306_Hole")
-    )
     (path "/00000000-0000-0000-0000-0000609f9aea"
       (reference "J1") (unit 1) (value " ") (footprint "Connector_JST:JST_SH_SM04B-SRSS-TB_1x04-1MP_P1.00mm_Horizontal")
@@
     )
     (path "/00000000-0000-0000-0000-000060e40d1e"
-      (reference "U2") (unit 1) (value "Display_Graphic_OLED_SSD1306_30-Pin") (footprint "Display:OLED-128O064D")
-    )
-  )
+      (reference "U2") (unit 1) (value "Display_Graphic_OLED_SSD1306_30-Pin") (footprint "CoreElectronics_Components:OLED-128O064D_reduced_paste")
+    )
+  )
